Commit message: gather together some files + add controlers to bullet + start of some data plot

File: pybullet/models/iRobot_simple/iRobot_simple.urdf (robot description, URDF)
Before this commit: robot iRobot, 6 links, 5 joints
Links:
- link base_footprint: geometry collision cylinder length=0.043000 radius=0.2000; visual cylinder length=0.043000 radius=0.2000
