Commit message: -

File: pybullet/models/iRobot/iRobot.urdf (robot description, URDF)
Before this commit: robot iRobot, 6 links, 5 joints
Links:
- link base_footprint: geometry collision mesh filename=meshes/create_body3.dae; visual mesh filename=meshes/create_body3.dae
- link laser: geometry collision mesh filename=meshes/hokuyo.obj scale=0.5 0.5 0.5 0.5; visual mesh filename=meshes/hokuyo.obj scale=0.5 0.5 0.5 0.5
Joints:
- joint hokuyo_joint: origin xyz=-0.08 0.0 0.085 rpy=0 0 0 -> xyz=-0.011 0.0 0.085 rpy=0 0 0

Commit message: -

File: pybullet/models/iRobot/iRobot.urdf (robot description, URDF)
Before this commit: robot iRobot, 6 links, 5 joints
Links:
- link base_footprint: mass None -> 2.234000
- link left_wheel_link: mass None -> 0.010000
- link right_wheel_link: mass None -> 0.010000

Commit message: small changes

File: pybullet/models/iRobot/iRobot.urdf (robot description, URDF)
Before this commit: robot iRobot, 6 links, 5 joints
Links:
- link base_footprint: mass 2.234000 -> 5.234000
- link left_wheel_link: mass 0.010000 -> 0.0100000

Commit message: experimental values - need further testing

File: pybullet/models/iRobot/iRobot.urdf (robot description, URDF)
Before this commit: robot iRobot, 6 links, 5 joints
Links:
- link left_wheel_link: mass 0.0100000 -> 0.34055
- link right_wheel_link: mass 0.010000 -> 0.34055

Commit message: changing robots and maps to be comparable
robots of same size, maps of same size, laser of same size and angle ( now in degree in bullet) .
Swap left and right wheel in bullet.
Changed the speed in bullet according to the real robot max velocity (500mm/s).
Following camera  now in the yml file (desactivate for better performance) Same as the GUI option.

File: pybullet/models/iRobot/iRobot.urdf (robot description, URDF)
Before this commit: robot iRobot, 6 links, 5 joints
Joints:
- joint hokuyo_joint: origin xyz=-0.011 0.0 0.085 rpy=0 0 0 -> xyz=0 0.0 0.085 rpy=0 0 0

Commit message: added bumpers in bullet, changed obs to be like fastsim, reorgonized folders and files, save and load HOF for FI+NV search, clean up

File: pybullet/models/iRobot/iRobot.urdf (robot description, URDF)
Before this commit: robot iRobot, 6 links, 5 joints
Links:
- added link left_bumper_laser, mass 0.0; visual box size=0.004712 0.01632 0.003089
- added link right_bumper_laser, mass 0.0; visual box size=0.004712 0.01632 0.003089
Joints:
- added joint left_bumper_laser_joint: type fixed, parent base_footprint, child left_bumper_laser, origin xyz=0.110948 0.122005 0.05 rpy=0. 0 0.872665, axis 0 0 1
- added joint right_bumper_laser_joint: type fixed, parent base_footprint, child right_bumper_laser, origin xyz=0.110948 -0.122005 0.05 rpy=0. 0 -0.872665, axis 0 0 1
- joint hokuyo_joint: origin xyz=0 0.0 0.085 rpy=0 0 0 -> xyz=0 0.0 0.09 rpy=0 0 0
